Commit message: Update joint limits in URDF and modify IK evaluation scripts for improved trajectory visualization. Adjusted limits for wrist, elbow, and shoulder joints in `so101_new_calib.urdf`. Changed line axis in `ik_eval_so101.py` from 'x' to 'z'. Enhanced `ik_play_in_placo.py` to visualize end-effector paths and save trajectory points for external plotting.

File: SO101/so101_new_calib.urdf (robot description, URDF)
Before this commit: robot so101_new_calib, 8 links, 7 joints
Joints:
- joint elbow_flex: limit lower=-1.69 upper=1.69 effort=10 velocity=10 -> lower=-1.71164 upper=1.71164 effort=10 velocity=10
- joint shoulder_lift: limit lower=-1.74533 upper=1.74533 effort=10 velocity=10 -> lower=-1.83347 upper=1.83347 effort=10 velocity=10
- joint shoulder_pan: limit lower=-1.91986 upper=1.91986 effort=10 velocity=10 -> lower=-2.03290 upper=2.03290 effort=10 velocity=10
- joint wrist_flex: limit lower=-1.65806 upper=1.65806 effort=10 velocity=10 -> lower=-1.79524 upper=1.79524 effort=10 velocity=10
- joint wrist_roll: limit lower=-2.74385 upper=2.84121 effort=10 velocity=10 -> lower=-2.94140 upper=2.94140 effort=10 velocity=10

Commit message: SO101 URDF: sync joint limits to calibrated ranges (deg→rad) for all 5 joints

File: SO101/so101_new_calib.urdf (robot description, URDF)
Before this commit: robot so101_new_calib, 8 links, 7 joints
Joints:
- joint elbow_flex: limit lower=-1.71164 upper=1.71164 effort=10 velocity=10 -> lower=-1.70309 upper=1.70309 effort=10 velocity=10
- joint shoulder_lift: limit lower=-1.83347 upper=1.83347 effort=10 velocity=10 -> lower=-1.97554 upper=1.97554 effort=10 velocity=10
- joint shoulder_pan: limit lower=-2.03290 upper=2.03290 effort=10 velocity=10 -> lower=-1.91795 upper=1.91795 effort=10 velocity=10
- joint wrist_flex: limit lower=-1.79524 upper=1.79524 effort=10 velocity=10 -> lower=-1.78828 upper=1.78828 effort=10 velocity=10
- joint wrist_roll: limit lower=-2.94140 upper=2.94140 effort=10 velocity=10 -> lower=-1.72543 upper=1.72543 effort=10 velocity=10

Commit message: SO101 URDF: update joint limits to latest calibrated ranges (deg→rad)

File: SO101/so101_new_calib.urdf (robot description, URDF)
Before this commit: robot so101_new_calib, 8 links, 7 joints
Joints:
- joint elbow_flex: limit lower=-1.70309 upper=1.70309 effort=10 velocity=10 -> lower=-1.55509 upper=1.55509 effort=10 velocity=10
- joint shoulder_lift: limit lower=-1.97554 upper=1.97554 effort=10 velocity=10 -> lower=-1.88426 upper=1.88426 effort=10 velocity=10
- joint shoulder_pan: limit lower=-1.91795 upper=1.91795 effort=10 velocity=10 -> lower=-1.91637 upper=1.91637 effort=10 velocity=10
- joint wrist_flex: limit lower=-1.78828 upper=1.78828 effort=10 velocity=10 -> lower=-1.80135 upper=1.80135 effort=10 velocity=10
- joint wrist_roll: limit lower=-1.72543 upper=1.72543 effort=10 velocity=10 -> lower=-1.64480 upper=1.64480 effort=10 velocity=10

Commit message: SO101 URDF: update joint limits for wrist, elbow, and shoulder joints to reflect new calibrated ranges

File: SO101/so101_new_calib.urdf (robot description, URDF)
Before this commit: robot so101_new_calib, 8 links, 7 joints
Joints:
- joint elbow_flex: limit lower=-1.55509 upper=1.55509 effort=10 velocity=10 -> lower=-1.72613 upper=1.72613 effort=10 velocity=10
- joint shoulder_lift: limit lower=-1.88426 upper=1.88426 effort=10 velocity=10 -> lower=-1.83975 upper=1.83975 effort=10 velocity=10
- joint shoulder_pan: limit lower=-1.91637 upper=1.91637 effort=10 velocity=10 -> lower=-1.95931 upper=1.95931 effort=10 velocity=10
- joint wrist_flex: limit lower=-1.80135 upper=1.80135 effort=10 velocity=10 -> lower=-1.80973 upper=1.80973 effort=10 velocity=10
- joint wrist_roll: limit lower=-1.64480 upper=1.64480 effort=10 velocity=10 -> lower=-1.69157 upper=1.69157 effort=10 velocity=10
