Commit message: Add ground truth end-effector trajectory extraction tools and URDF model
- Introduced `extract_gt_ee_trajectories.py` for extracting and transforming end-effector trajectories from the LeRobotDataset, saving them as CSV files.
- Added README.md documentation for the trajectory extraction tool, detailing usage, output format, and arguments.
- Included a new URDF model file `piper_description_old.urdf` for the Piper robot, defining its structure and joints.
- Created `piper_print_state.py` to read and print the state of the Piper robot without enabling motors, providing joint angles, end-effector pose, and gripper state.

File: traj_execution_test/piper_mujoco/piper_description_old.urdf (robot description, URDF)
Before this commit: robot piper_description, 10 links, 9 joints
Links:
- added link gripper_base, mass 0.45; collision mesh filename=meshes/gripper_base.STL; visual mesh filename=meshes/gripper_base.STL
- link base_link: mass 0.162352169522719 -> 1.02; geometry collision mesh filename=meshes/base_link.STL; visual mesh filename=meshes/base_link.STL
- link link1: mass 0.0978679932242825 -> 0.71; geometry collision mesh filename=meshes/link1.STL; visual mesh filename=meshes/link1.STL
- link link2: mass 0.289571136953082 -> 1.17; geometry collision mesh filename=meshes/link2.STL; visual mesh filename=meshes/link2.STL
- link link3: mass 0.290583247455324 -> 0.5; geometry collision mesh filename=meshes/link3.STL; visual mesh filename=meshes/link3.STL
- link link4: mass 0.127087348341362 -> 0.38; geometry collision mesh filename=meshes/link4.STL; visual mesh filename=meshes/link4.STL
- link link5: mass 0.144711209371719 -> 0.383; geometry collision mesh filename=meshes/link5.STL; visual mesh filename=meshes/link5.STL
- link link6: mass 0.150196458571266 -> 0.007; geometry collision mesh filename=meshes/link6.STL; visual mesh filename=meshes/link6.STL
- link link7: mass 0.0264822500394006 -> 0.025; geometry collision mesh filename=meshes/link7.STL; visual mesh filename=meshes/link7.STL
- link link8: mass 0.0264822490707451 -> 0.025; geometry collision mesh filename=meshes/link8.STL; visual mesh filename=meshes/link8.STL
Joints:
- added joint joint6_to_gripper_base: type fixed, parent link6, child gripper_base, origin xyz=0 0 0 rpy=0 0 0
- joint ee_joint: origin xyz=0 0 0.13 rpy=1.5707963 -1.5707963 0 -> xyz=0 0 0.135 rpy=-1.5707963 0 -1.5707963
- joint joint1: limit lower=-2.618 upper=2.618 effort=100 velocity=3 -> lower=-2.618 upper=2.168 effort=100 velocity=5; origin xyz=0 0 0.123 rpy=0 0 -1.5708 -> xyz=0 0 0.123 rpy=0 0 0
- joint joint2: limit lower=0 upper=3.14 effort=100 velocity=3 -> lower=0 upper=3.14 effort=100 velocity=5; origin xyz=0 0 0 rpy=1.5708 -0.10095 -1.5708 -> xyz=0 0 0 rpy=1.5708 -0.10095 -3.1416
- joint joint3: limit lower=-2.967 upper=0 effort=100 velocity=3 -> lower=-2.967 upper=0 effort=100 velocity=5; origin xyz=0.28503 0 0 rpy=0 0 1.3826 -> xyz=0.28503 0 0 rpy=0 0 -1.759
- joint joint4: limit lower=-1.832 upper=1.832 effort=100 velocity=3 -> lower=-1.745 upper=1.745 effort=100 velocity=5; origin xyz=0.021984 0.25075 0 rpy=-1.5708 0 0 -> xyz=-0.021984 -0.25075 0 rpy=1.5708 0 0
- joint joint5: limit lower=-1.22 upper=1.22 effort=100 velocity=3 -> lower=-1.22 upper=1.22 effort=100 velocity=5; origin xyz=0 0 0 rpy=1.5708 0 0 -> xyz=0 0 0 rpy=-1.5708 0 0
- joint joint6: axis 0 0 -1 -> 0 0 1; limit lower=-3.14 upper=3.14 effort=100 velocity=3 -> lower=-2.0944 upper=2.0944 effort=100 velocity=3; origin xyz=0 0.091 0.0014165 rpy=-1.5708 -1.5708 0 -> xyz=8.8259E-05 -0.091 0 rpy=1.5708 0 0
- joint joint7: axis 0 0 -1 -> 0 0 1; limit lower=0 upper=0.04 effort=100 velocity=1 -> lower=0 upper=0.035 effort=10 velocity=1; origin xyz=0 0 0.13503 rpy=1.5708 0 1.5708 -> xyz=0 0 0.1358 rpy=1.5708 0 0; parent link6 -> gripper_base
- joint joint8: axis 0 0 1 -> 0 0 -1; limit lower=-0.04 upper=0 effort=100 velocity=1 -> lower=-0.035 upper=0 effort=10 velocity=1; origin xyz=0 0 0.13503 rpy=-1.5708 0 1.5708 -> xyz=0 0 0.1358 rpy=1.5708 0 -3.1416; parent link6 -> gripper_base

Commit message: fix: update URDF path to use the correct file for Piper robot

File: traj_execution_test/piper_mujoco/piper_description_old.urdf (robot description, URDF)
Before this commit: robot piper, 11 links, 10 joints
Links:
- removed link gripper_base
Joints:
- removed joint joint6_to_gripper_base
- joint joint7: parent gripper_base -> link6
- joint joint8: parent gripper_base -> link6
