Commit message: feat: add --plot-tcp-traj mode and ORB-SLAM trajectory visualization script
- Add --plot-tcp-traj flag to piper_mujoco_traj_test.py: plots TCP trajectory
  using Placo FK only, no MuJoCo launched
- Add visualize_orb_traj.py: visualize ORB-SLAM camera trajectories with
  XY/XZ/YZ + 3D + xyz-vs-steps plot, and --video flag for h265 mp4 from color*.png
- Update URDF with camera_link frame chain

Co-Authored-By: Claude Opus 4.6 <noreply@anthropic.com>

File: traj_execution_test/piper_mujoco/piper_description.urdf (robot description, URDF)
Before this commit: robot piper_description, 10 links, 9 joints
Links:
- added link camera_dummy_link
- added link camera_link; visual box size=0.01 0.05 0.02
- link ee_link: geometry 
Joints:
- added joint camera_dummy_joint: type fixed, parent link6, child camera_dummy_link, origin xyz=0 0.07 0.03 rpy=-1.5707963 -1.5707963 0
- added joint camera_joint: type fixed, parent camera_dummy_link, child camera_link, origin xyz=0 0 0 rpy=0 0.25 0
- joint ee_joint: origin xyz=0 0 0.13 rpy=1.5707963 -1.5707963 0 -> xyz=0 0 0 rpy=0 0 0; parent link6 -> camera_link
